File: Schematics/Schematic.kicad_sch (KiCad schematic)
At the start: 27 parts, among them J1 Audio Input, J2 Audio Output, J3 +9V, U1 MCP6002, U2 LM78L05, U3 LD33CV

Commit message: Filter fixes, electric circuit fix (KiCad updated)
Parts:
- R3: value 1k -> 1M
- R4, R5, R6, R7: value 20k -> 1M
Changed lines of the file:
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@@
 			)
 		)
-		(property "Value" "20k"
+		(property "Value" "1M"
 			(at 76.2 35.5599 0)
 			(effects
@@
 			)
 		)
-		(property "Value" "20k"
+		(property "Value" "1M"
 			(at 69.85 104.1399 0)
 			(effects
@@
 			)
 		)
-		(property "Value" "1k"
+		(property "Value" "1M"
 			(at 60.96 38.1 90)
 			(effects
@@
 			)
 		)
-		(property "Value" "20k"
+		(property "Value" "1M"
 			(at 67.31 88.8999 0)
 			(effects
@@
 			)
 		)
-		(property "Value" "20k"
+		(property "Value" "1M"
 			(at 71.12 50.7999 0)
 			(effects

Commit message: Schematics work
Parts:
- added D2: LED, symbol Device:LED
- added R10, R11: 10K, symbol Device:R
- added R9: 330, symbol Device:R
- added RV1, RV2, RV3, RV4: 10K, symbol Device:R_Potentiometer
- added SW1, SW2, SW3, SW4: SW_Push, symbol Switch:SW_Push
- added SW5: Active / passive pickup switch, Button_Switch_SMD:Nidec_Copal_CAS-120A, symbol Switch:SW_Nidec_CAS-120A1
- added U4: ~, symbol Teensy:Teensy 4.1 + Audio Shield rev D
Connections:
- net +3.3V: now also RV1.1, RV2.1, RV3.1, RV4.1, SW1.1, SW2.1, SW3.1, SW4.1
- net +5V: now also U4. (33)
- net GND: now also R11.2, R9.1, RV1.3, RV2.3, RV3.3, RV4.3, U4. (33)
- net Line-in: now also SW5.2 (B), U4. (33); no longer U1.2 (-)
- net Line-out: now also U4. (33)
- new net: D2.1 (K), R9.2
- new net: R10.2, R11.1, SW5.3 (A), U1.2 (-)
- new net: R10.1, SW5.1 (C)
- new net EFFECT EN: SW4.2, U4. (33)
- new net EFFECT L SEL: SW2.2, U4. (33)
- new net EFFECT R SEL: SW3.2, U4. (33)
- new net MODIFY BUTTON: SW1.2, U4. (33)
- new net MODIFY LED: D2.2 (A), U4. (33)
- new net PAR1: RV1.2, U4. (33)
- new net PAR2: RV2.2, U4. (33)
- new net PAR3: RV3.2, U4. (33)
- new net PAR4: RV4.2, U4. (33)
Other:
- moved on the sheet: C1, C10, C11, C12, C2, C3, C4, C5, C6, C7, C8, C9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
